Commit message: dd

File: urdf/robot.urdf.xacro (robot description, xacro)
@@ -21,4 +21,58 @@
     </inertial>
   </link>
+  <!-- Left Wheel -->
+  <link name="left_wheel">
+    <visual>
+      <geometry>
+        <cylinder radius="0.05" length="0.04"/>
+      </geometry>
+      <material name="black">
+        <color rgba="0 0 0 1"/>
+      </material>
+    </visual>
+    <collision>
+      <geometry>
+        <cylinder radius="0.05" length="0.04"/>
+      </geometry>
+    </collision>
+    <inertial>
+      <mass value="0.1"/>
+      <inertia ixx="0.00001" ixy="0" ixz="0" iyy="0.00001" iyz="0" izz="0.00001"/>
+    </inertial>
+  </link>
+  <!-- Right Wheel -->
+  <link name="right_wheel">
+    <visual>
+      <geometry>
+        <cylinder radius="0.05" length="0.04"/>
+      </geometry>
+      <material name="black">
+        <color rgba="0 0 0 1"/>
+      </material>
+    </visual>
+    <collision>
+      <geometry>
+        <cylinder radius="0.05" length="0.04"/>
+      </geometry>
+    </collision>
+    <inertial>
+      <mass value="0.1"/>
+      <inertia ixx="0.00001" ixy="0" ixz="0" iyy="0.00001" iyz="0" izz="0.00001"/>
+    </inertial>
+  </link>
+  <!-- Left Wheel Joint -->
+  <joint name="left_wheel_joint" type="continuous">
+    <parent link="base_link"/>
+    <child link="left_wheel"/>
+    <origin xyz="0 0.12 -0.025" rpy="-1.5707 0 0"/>
+    <axis xyz="0 0 1"/>
+  </joint>
+  <!-- Right Wheel Joint -->
+  <joint name="right_wheel_joint" type="continuous">
+    <parent link="base_link"/>
+    <child link="right_wheel"/>
+    <origin xyz="0 -0.12 -0.025" rpy="-1.5707 0 0"/>
+    <axis xyz="0 0 1"/>
+  </joint>
   <!-- Laser Link -->
   <link name="laser">

Commit message: ss

File: urdf/robot.urdf.xacro (robot description, xacro)
@@ -81,7 +81,5 @@
         <cylinder radius="0.03" length="0.05"/>
       </geometry>
-      <material name="black">
-        <color rgba="0 0 0 1"/>
-      </material>
+      <material name="black"/>
     </visual>
     <collision>
@@ -112,11 +110,10 @@
     </plugin>
   </gazebo>
-  <!-- Laser plugin -->
+  <!-- Gazebo plugins for laser -->
   <gazebo reference="laser">
-    <sensor type="gpu_ray" name="rplidar">
-      <pose>0 0 0 0 0 0</pose>
-      <visualize>true</visualize>
+    <sensor name='gpu_lidar' type='gpu_lidar'>
+      <topic>lidar</topic>
       <update_rate>10</update_rate>
-      <ray>
+      <lidar>
         <scan>
           <horizontal>
@@ -132,9 +129,10 @@
           <resolution>0.01</resolution>
         </range>
-      </ray>
-      <plugin filename="gz-sim-gpu-lidar-system"
-              name="gz::sim::systems::GpuLidar">
-        <topic>/lidar</topic>
-        <frame_name>laser</frame_name>
+      </lidar>
+      <visualize>true</visualize>
+      <always_on>1</always_on>
+      <plugin name='gpu_lidar' filename='gz-sim-gpu-lidar-system'>
+        <gz_frame_id>laser</gz_frame_id>
+        <topic>lidar</topic>
       </plugin>
     </sensor>
